Commit message: 提交 feat-gps-20260226 分支的修改

File: LIO-SAM_MID360_ROS2_PKG/ros2/src/livox_gazebo_ros2_gpu_simulation/urdf/my_robot/my_robot.xacro (robot description, xacro)
@@ -94,9 +94,4 @@
 <xacro:my_robot_ros2_control_planar />   <!-- 如果gazebo_control更改名字，请修改此处 -->
 <xacro:gazebo_sensor_plugin />
-<!-- gazebo_ros2_control plugin -->
-<gazebo>
-  <plugin name="gazebo_ros2_control" filename="libgazebo_ros2_control.so">
-    <parameters>/home/ywj/dog_slam/LIO-SAM_MID360_ROS2_PKG/ros2/install/livox_gazebo_ros2_gpu_simulation/share/livox_gazebo_ros2_gpu_simulation/config/myrobot_ros2_controller.yaml</parameters>
-  </plugin>
-</gazebo>
+<!-- gazebo_ros2_control plugin - removed to avoid crashes -->
 </robot>

File: LIO-SAM_MID360_ROS2_PKG/ros2/src/livox_gazebo_ros2_gpu_simulation/urdf/my_robot/plugins/gazebo_control_plugin.xacro (robot description, xacro)
@@ -3,42 +3,4 @@
    <!-- 按需更改 名字 -->
     <xacro:macro name="my_robot_ros2_control_planar">
-        <ros2_control name="MyRobotPlanarSystem" type="system">
-            <hardware>
-                <plugin>gazebo_ros2_control/GazeboSystem</plugin>
-            </hardware>
-            <!-- 定义关节接口 -->
-            <joint name="behind_left_wheel_joint">
-                <command_interface name="velocity">
-                    <param name="min">-10</param>
-                    <param name="max">10</param>
-                </command_interface>
-                <state_interface name="position"/>
-                <state_interface name="velocity"/>
-            </joint>
-            <joint name="behind_right_wheel_joint">
-                <command_interface name="velocity">
-                    <param name="min">-10</param>
-                    <param name="max">10</param>
-                </command_interface>
-                <state_interface name="position"/>
-                <state_interface name="velocity"/>
-            </joint>
-            <joint name="ahead_left_wheel_joint">
-                <command_interface name="velocity">
-                    <param name="min">-10</param>
-                    <param name="max">10</param>
-                </command_interface>
-                <state_interface name="position"/>
-                <state_interface name="velocity"/>
-            </joint>
-            <joint name="ahead_right_wheel_joint">
-                <command_interface name="velocity">
-                    <param name="min">-10</param>
-                    <param name="max">10</param>
-                </command_interface>
-                <state_interface name="position"/>
-                <state_interface name="velocity"/>
-            </joint>
-        </ros2_control>
         <gazebo>
         <!-- libgazebo_ros_planar_move.so 是 平面移动插件 -->

File: LIO-SAM_MID360_ROS2_PKG/ros2/src/livox_gazebo_ros2_gpu_simulation/urdf/my_robot/sensor/mid360_cpu.xacro (robot description, xacro)
@@ -26,5 +26,5 @@
         <origin xyz="0.025 -0.0265 -0.025" rpy="${pi/2} 0 ${pi}"/>
         <geometry>
-          <mesh filename="package://livox_gazebo_ros2_gpu_simulation/meshes/mid360.stl" scale="0.0008 0.0008 0.0008"/>
+          <mesh filename="file:///home/crazytree/ros_ws/dog_slam/LIO-SAM_MID360_ROS2_PKG/ros2/src/livox_gazebo_ros2_gpu_simulation/meshes/mid-360-scaled.dae" scale="1 1 1"/>
         </geometry>
       </visual>
@@ -32,5 +32,5 @@
     <origin xyz="0.025 -0.0265 -0.025" rpy="${pi/2} 0 ${pi}"/>
     <geometry>
-      <mesh filename="package://livox_gazebo_ros2_gpu_simulation/meshes/mid360.stl" scale="0.0008 0.0008 0.0008"/>
+      <mesh filename="file:///home/crazytree/ros_ws/dog_slam/LIO-SAM_MID360_ROS2_PKG/ros2/src/livox_gazebo_ros2_gpu_simulation/meshes/mid-360-scaled.dae" scale="1 1 1"/>
     </geometry>
   </collision>
